Commit message: Imported the CAD model via Blender. Somewhat works with MoveIt now, but start state wrong

File: urdf/arm.xacro (robot description, xacro)
@@ -18,6 +18,10 @@
     <xacro:property name="offset_gripper" value="0.01" />
     <xacro:property name="lim_eff" value="300" />
-    <xacro:property name="lim_low" value="-2.78539816339" />
-    <xacro:property name="lim_up" value="2.78539816339" />
+    <xacro:property name="lim_low_1" value="${-pi * 1/3}" />
+    <xacro:property name="lim_up_1" value="${pi * 2/3}" />
+    <xacro:property name="lim_low_2" value="-2.9698" />
+    <xacro:property name="lim_up_2" value="1.18" />
+    <xacro:property name="lim_low_4" value="${-pi/2}" />
+    <xacro:property name="lim_up_4" value="${pi/2}" />
     <xacro:property name="lim_vel" value="1.571" />
     <xacro:macro name="box_inertia" params="m x y z">
@@ -34,230 +38,161 @@
     </material>
     <xacro:macro name="arm" params="parent translateX translateY translateZ">
-        <joint name="joint_base" type="revolute">
+        <!--  Link 0: rotating base  -->
+        <joint name="joint0" type="continuous">
             <parent link="${parent}"/>
             <child link="link0"/>
             <origin rpy="0 0 0" xyz="${translateX} ${translateY} ${translateZ}"/>
             <axis xyz="0 0 1"/>
-            <limit effort="${lim_eff}" lower="${lim_low}" upper="${lim_up}" velocity="${lim_vel}"/>
+            <limit effort="${lim_eff}" velocity="${lim_vel}"/>
         </joint>
         <link name="link0">
             <collision>
+                <origin rpy="0 0 0" xyz="0 0 0"/>
+                <geometry>
+                    <mesh filename="package://rover_arm/meshes/Coll_Link0.stl"/>
+                </geometry>
+            </collision>
+            <visual>
+                <origin rpy="0 0 0" xyz="0 0 0"/>
+                <geometry>
+                    <mesh filename="package://rover_arm/meshes/Link0.dae"/>
+                </geometry>
+                <material name="orange"/>
+            </visual>
+            <inertial>
                 <origin rpy="0 0 0" xyz="0 0 ${link0_len/2}"/>
-                <geometry>
-                    <cylinder length="${link0_len}" radius="${link0_rad}"/>
-                </geometry>
-            </collision>
-            <visual>
-                <origin rpy="0 0 0" xyz="0 0 ${link0_len/2}"/>
-                <geometry>
-                    <cylinder length="${link0_len}" radius="${link0_rad}"/>
-                </geometry>
-                <material name="orange"/>
-            </visual>
-            <inertial>
-                <origin rpy="0 0 0" xyz="0 0 ${link0_len/2}"/>
                 <mass value="1"/>
                 <cylinder_inertia m="1" r="${link0_rad}" h="${link0_len}" />
             </inertial>
         </link>
-        <joint name="joint0" type="revolute">
+        <!--  Link 1: up/down arm segment 1  -->
+        <joint name="joint1" type="revolute">
             <parent link="link0"/>
             <child link="link1"/>
-            <origin rpy="0 0 0" xyz="0 0 ${link0_len}"/>
-            <axis xyz="0 1 0"/>
-            <limit effort="${lim_eff}" lower="${lim_low}" upper="${lim_up}" velocity="${lim_vel}"/>
+                <origin rpy="0 0 0" xyz="0 0.1 0.1"/>
+            <axis xyz="1 0 0"/>
+            <limit effort="${lim_eff}" lower="${lim_low_1}" upper="${lim_up_1}" velocity="${lim_vel}"/>
         </joint>
         <link name="link1">
             <collision>
+                <origin rpy="0 0 0" xyz="0 0 0"/>
+                <geometry>
+                    <mesh filename="package://rover_arm/meshes/Coll_Link1.stl"/>
+                </geometry>
+            </collision>
+            <visual>
+                <origin rpy="0 0 0" xyz="0 0 0"/>
+                <geometry>
+                    <mesh filename="package://rover_arm/meshes/Link1.dae"/>
+                </geometry>
+                <material name="black"/>
+            </visual>
+            <inertial>
                 <origin rpy="0 0 0" xyz="0 0 ${link1_len/2}"/>
-                <geometry>
-                    <box size="${link1_width} ${link1_width} ${link1_len}"/>
-                </geometry>
-            </collision>
-            <visual>
-                <origin rpy="0 0 0" xyz="0 0 ${link1_len/2}"/>
-                <geometry>
-                    <box size="${link1_width} ${link1_width} ${link1_len}"/>
-                </geometry>
-                <material name="black"/>
-            </visual>
-            <inertial>
-                <origin rpy="0 0 0" xyz="0 0 ${link1_len/2}"/>
                 <mass value="1"/>
                 <box_inertia m="1" x="${link1_width}" y="${link1_width}" z="${link1_len}" />
             </inertial>
         </link>
-        <joint name="joint1" type="revolute">
+        <!--  Link 2: up/down arm segment 2  -->
+        <joint name="joint2" type="revolute">
             <parent link="link1"/>
             <child link="link2"/>
-            <origin rpy="0 0 0" xyz="0 0 ${link1_len}"/>
-            <axis xyz="0 1 0"/>
-            <limit effort="${lim_eff}" lower="${lim_low}" upper="${lim_up}" velocity="${lim_vel}"/>
+                <origin rpy="0 0 0" xyz="0 0.3 0"/>
+            <axis xyz="1 0 0"/>
+            <limit effort="${lim_eff}" lower="${lim_low_2}" upper="${lim_up_2}" velocity="${lim_vel}"/>
         </joint>
         <link name="link2">
             <collision>
+                <origin rpy="0 0 0" xyz="0 0 0"/>
+                <geometry>
+                    <mesh filename="package://rover_arm/meshes/Coll_Link2.stl"/>
+                </geometry>
+            </collision>
+            <visual>
+                <origin rpy="0 0 0" xyz="0 0 0"/>
+                <geometry>
+                    <mesh filename="package://rover_arm/meshes/Link2.dae"/>
+                </geometry>
+                <material name="orange"/>
+            </visual>
+            <inertial>
                 <origin rpy="0 0 0" xyz="0 0 ${link2_len/2}"/>
-                <geometry>
-                    <box size="${link2_width} ${link2_width} ${link2_len}"/>
-                </geometry>
-            </collision>
-            <visual>
-                <origin rpy="0 0 0" xyz="0 0 ${link2_len/2}"/>
-                <geometry>
-                    <box size="${link2_width} ${link2_width} ${link2_len}"/>
-                </geometry>
-                <material name="orange"/>
-            </visual>
-            <inertial>
-                <origin rpy="0 0 0" xyz="0 0 ${link2_len/2}"/>
                 <mass value="1"/>
                 <box_inertia m="1" x="${link2_width}" y="${link2_width}" z="${link2_len}" />
             </inertial>
         </link>
-        <joint name="joint2" type="revolute">
+        <!--  Link 3: swivel forward  -->
+        <joint name="joint3" type="continuous">
             <parent link="link2"/>
             <child link="link3"/>
-            <origin rpy="0 0 0" xyz="0 0 ${link2_len}"/>
-            <axis xyz="0 0 1"/>
-            <limit effort="${lim_eff}" lower="${lim_low}" upper="${lim_up}" velocity="${lim_vel}"/>
+                <origin rpy="0 0 0" xyz="0 0.1993 0.1"/>
+            <axis xyz="0 1 0"/>
+            <limit effort="${lim_eff}" velocity="${lim_vel}"/>
         </joint>
         <link name="link3">
-            <collision>
-                <origin rpy="0 0 0" xyz="0 0 ${link3_len/2}"/>
-                <geometry>
-                    <box size="${link3_width} ${link3_width} ${link3_len}"/>
-                </geometry>
-            </collision>
-            <visual>
-                <origin rpy="0 0 0" xyz="0 0 ${link3_len/2}"/>
-                <geometry>
-                    <box size="${link3_width} ${link3_width} ${link3_len}"/>
+            <visual>
+                <origin rpy="0 0 0" xyz="0 0 0"/>
+                <geometry>
+                    <mesh filename="package://rover_arm/meshes/Link3.dae"/>
                 </geometry>
                 <material name="black"/>
             </visual>
             <inertial>
-                <origin rpy="0 0 0" xyz="0 0 ${link3_len/2}"/>
+                <origin rpy="0 0 0" xyz="0 0 0"/>
                 <mass value="1"/>
                 <box_inertia m="1" x="${link3_width}" y="${link3_width}" z="${link3_len}" />
             </inertial>
         </link>
-        <joint name="joint3" type="revolute">
+        <!--  Link 4: swivel up/down  -->
+        <joint name="joint4" type="revolute">
             <parent link="link3"/>
             <child link="link4"/>
-            <origin rpy="0 0 0" xyz="0 0 ${link3_len}"/>
+                <origin rpy="0 0 0" xyz="0.019276 0.052499 0"/>
+            <axis xyz="1 0 0"/>
+            <limit effort="${lim_eff}" lower="${lim_low_4}" upper="${lim_up_4}" velocity="${lim_vel}"/>
+        </joint>
+        <link name="link4">
+            <visual>
+                <origin rpy="0 0 0" xyz="0 0 0"/>
+                <geometry>
+                    <mesh filename="package://rover_arm/meshes/Link4.dae"/>
+                </geometry>
+                <material name="orange"/>
+            </visual>
+            <inertial>
+                <origin rpy="0 0 0" xyz="0 0 0"/>
+                <mass value="1"/>
+                <box_inertia m="1" x="${link4_width}" y="${link4_width}" z="${link4_len}" />
+            </inertial>
+        </link>
+        <!--  Hand and swivel forward  -->
+        <joint name="joint_hand" type="continuous">
+            <parent link="link4"/>
+            <child link="link_hand"/>
+                <origin rpy="0 0 0" xyz="-0.019288 0.03 0"/>
             <axis xyz="0 1 0"/>
-            <limit effort="${lim_eff}" lower="${lim_low}" upper="${lim_up}" velocity="${lim_vel}"/>
-        </joint>
-        <link name="link4">
-            <collision>
-                <origin rpy="0 0 0" xyz="0 0 ${link4_len/2}"/>
-                <geometry>
-                    <box size="${link4_width} ${link4_width} ${link4_len}"/>
-                </geometry>
-            </collision>
-            <visual>
-                <origin rpy="0 0 0" xyz="0 0 ${link4_len/2}"/>
-                <geometry>
-                    <box size="${link4_width} ${link4_width} ${link4_len}"/>
-                </geometry>
-                <material name="orange"/>
-            </visual>
-            <inertial>
-                <origin rpy="0 0 0" xyz="0 0 ${link4_len/2}"/>
-                <mass value="1"/>
-                <box_inertia m="1" x="${link4_width}" y="${link4_width}" z="${link4_len}" />
-            </inertial>
-        </link>
-        <joint name="joint4" type="revolute">
-            <parent link="link4"/>
-            <child link="link5"/>
-            <origin rpy="0 0 0" xyz="0 0 ${link4_len}"/>
-            <axis xyz="0 0 1"/>
-            <limit effort="${lim_eff}" lower="${lim_low}" upper="${lim_up}" velocity="${lim_vel}"/>
-        </joint>
-        <link name="link5">
-            <collision>
+            <limit effort="${lim_eff}" velocity="${lim_vel}"/>
+        </joint>
+        <link name="link_hand">
+            <collision>
+                <origin rpy="0 0 0" xyz="0 0 0"/>
+                <geometry>
+                    <mesh filename="package://rover_arm/meshes/Coll_Hand.stl"/>
+                </geometry>
+            </collision>
+            <visual>
+                <origin rpy="0 0 0" xyz="0 0 0"/>
+                <geometry>
+                    <mesh filename="package://rover_arm/meshes/Hand.dae"/>
+                </geometry>
+                <material name="black"/>
+            </visual>
+            <inertial>
                 <origin rpy="0 0 0" xyz="0 0 ${link5_len/2}"/>
-                <geometry>
-                    <box size="${link5_width} ${link5_width} ${link5_len}"/>
-                </geometry>
-            </collision>
-            <visual>
-                <origin rpy="0 0 0" xyz="0 0 ${link5_len/2}"/>
-                <geometry>
-                    <box size="${link5_width} ${link5_width} ${link5_len}"/>
-                </geometry>
-                <material name="black"/>
-            </visual>
-            <inertial>
-                <origin rpy="0 0 0" xyz="0 0 ${link5_len/2}"/>
                 <mass value="1"/>
                 <box_inertia m="1" x="${link5_width}" y="${link5_width}" z="${link5_len}" />
             </inertial>
         </link>
-        <joint name="joint5" type="revolute">
-            <parent link="link5"/>
-            <child link="gripper_left"/>
-            <origin rpy="0 0 0" xyz="0 ${offset_gripper} ${link5_len}"/>
-            <axis xyz="1 0 0"/>
-            <limit effort="${lim_eff}" lower="${lim_low}" upper="${lim_up}" velocity="${lim_vel}"/>
-        </joint>
-        <joint name="joint6" type="revolute">
-            <parent link="link5"/>
-            <child link="gripper_right"/>
-            <origin rpy="0 0 0" xyz="0 -${offset_gripper} ${link5_len}"/>
-            <axis xyz="1 0 0"/>
-            <limit effort="${lim_eff}" lower="${lim_low}" upper="${lim_up}" velocity="${lim_vel}"/>
-        </joint>
-        <link name="gripper_left">
-            <collision>
-                <origin rpy="0 0 0" xyz="0 0 ${gripper_len/2}"/>
-                <geometry>
-                    <cylinder length="${gripper_len}" radius="${gripper_rad}"/>
-                </geometry>
-            </collision>
-            <visual>
-                <origin rpy="0 0 0" xyz="0 0 ${gripper_len/2}"/>
-                <geometry>
-                    <cylinder length="${gripper_len}" radius="${gripper_rad}"/>
-                </geometry>
-                <material name="orange"/>
-            </visual>
-            <inertial>
-                <origin rpy="0 0 0" xyz="0 0 ${gripper_len/2}"/>
-                <mass value="1"/>
-                <cylinder_inertia m="1" r="${gripper_rad}" h="${gripper_len}" />
-            </inertial>
-        </link>
-        <link name="gripper_right">
-            <collision>
-                <origin rpy="0 0 0" xyz="0 0 ${gripper_len/2}"/>
-                <geometry>
-                    <cylinder length="${gripper_len}" radius="${gripper_rad}"/>
-                </geometry>
-            </collision>
-            <visual>
-                <origin rpy="0 0 0" xyz="0 0 ${gripper_len/2}"/>
-                <geometry>
-                    <cylinder length="${gripper_len}" radius="${gripper_rad}"/>
-                </geometry>
-                <material name="orange"/>
-            </visual>
-            <inertial>
-                <origin rpy="0 0 0" xyz="0 0 ${gripper_len/2}"/>
-                <mass value="1"/>
-                <cylinder_inertia m="1" r="${gripper_rad}" h="${gripper_len}" />
-            </inertial>
-        </link>
         <!-- Transmission is important to link the joint and the controller -->
-        <transmission name="joint_base_trans">
-            <type>transmission_interface/SimpleTransmission</type>
-            <joint name="joint_base">
-                <hardwareInterface>hardware_interface/EffortJointInterface</hardwareInterface>
-            </joint>
-            <actuator name="joint_base_motor">
-                <mechanicalReduction>1</mechanicalReduction>
-            </actuator>
-        </transmission>
         <transmission name="joint0_trans">
             <type>transmission_interface/SimpleTransmission</type>
@@ -305,22 +240,13 @@
             </actuator>
         </transmission>
-        <transmission name="joint5_trans">
-            <type>transmission_interface/SimpleTransmission</type>
-            <joint name="joint5">
-                <hardwareInterface>hardware_interface/EffortJointInterface</hardwareInterface>
-            </joint>
-            <actuator name="joint5_motor">
-                <mechanicalReduction>1</mechanicalReduction>
-            </actuator>
-        </transmission>
-        <transmission name="joint6_trans">
-            <type>transmission_interface/SimpleTransmission</type>
-            <joint name="joint6">
-                <hardwareInterface>hardware_interface/EffortJointInterface</hardwareInterface>
-            </joint>
-            <actuator name="joint6_motor">
-                <mechanicalReduction>1</mechanicalReduction>
-            </actuator>
-            </transmission>
+        <transmission name="joint_hand_trans">
+            <type>transmission_interface/SimpleTransmission</type>
+            <joint name="joint_hand">
+                <hardwareInterface>hardware_interface/EffortJointInterface</hardwareInterface>
+            </joint>
+            <actuator name="joint_hand_motor">
+                <mechanicalReduction>1</mechanicalReduction>
+            </actuator>
+        </transmission>
     </xacro:macro>
 </robot>

File: urdf/testarm.xacro (robot description, xacro)
@@ -33,5 +33,4 @@
       <plugin name="joint_state_publisher" filename="libgazebo_ros_joint_state_publisher.so">
          <jointName>
-            joint_base,
             joint0,
             joint1,
@@ -39,6 +38,5 @@
             joint3,
             joint4,
-            joint5,
-            joint6
+            joint_hand
          </jointName>
          <robotNameSpace>/</robotNameSpace>
