Commit message: better (still not good) pid parameters, less flailing around

File: urdf/arm.xacro (robot description, xacro)
@@ -2,4 +2,17 @@
 <robot name="arm"
     xmlns:xacro="http://www.ros.org/wiki/xacro">
+    <!-- com = center of mass -->
+    <xacro:property name="link0_com" value="0 0.1 0.05" />
+    <xacro:property name="link0_mass" value="3" />
+    <xacro:property name="link1_com" value="0 0.15 0" />
+    <xacro:property name="link1_mass" value="5" />
+    <xacro:property name="link2_com" value="0 0.1 0.1" />
+    <xacro:property name="link2_mass" value="2" />
+    <xacro:property name="link3_com" value="0 0.02 0" />
+    <xacro:property name="link3_mass" value="0.2" />
+    <xacro:property name="link4_com" value="-0.02 0 0" />
+    <xacro:property name="link4_mass" value="0.3" />
+    <xacro:property name="link_hand_com" value="0 0.05 0.02" />
+    <xacro:property name="link_hand_mass" value="1" />
     <xacro:property name="link0_len" value="0.1" />
     <xacro:property name="link0_rad" value="0.1" />
@@ -17,5 +30,5 @@
     <xacro:property name="gripper_rad" value="0.01" />
     <xacro:property name="offset_gripper" value="0.01" />
-    <xacro:property name="lim_eff" value="300" />
+    <xacro:property name="lim_eff" value="3000" />
     <xacro:property name="lim_low_1" value="${-pi * 1/3}" />
     <xacro:property name="lim_up_1" value="${pi * 2/3}" />
@@ -56,21 +69,22 @@
                 <origin rpy="0 0 0" xyz="0 0 0"/>
                 <geometry>
-                    <mesh filename="package://rover_arm/meshes/Link0.dae"/>
+                    <mesh filename="package://rover_arm/meshes/Coll_Link0.stl"/>
                 </geometry>
                 <material name="orange"/>
             </visual>
             <inertial>
-                <origin rpy="0 0 0" xyz="0 0 ${link0_len/2}"/>
-                <mass value="1"/>
-                <cylinder_inertia m="1" r="${link0_rad}" h="${link0_len}" />
+                <origin rpy="0 0 0" xyz="${link0_com}"/>
+                <mass value="${link0_mass}"/>
+                <cylinder_inertia m="${link0_mass}" r="${link0_rad}" h="0.5" />
             </inertial>
         </link>
         <!--  Link 1: up/down arm segment 1  -->
-        <joint name="joint1" type="revolute">
+        <joint name="joint1" type="continuous">
             <parent link="link0"/>
             <child link="link1"/>
                 <origin rpy="0 0 0" xyz="0 0.1 0.1"/>
             <axis xyz="1 0 0"/>
-            <limit effort="${lim_eff}" lower="${lim_low_1}" upper="${lim_up_1}" velocity="${lim_vel}"/>
+            <limit effort="${lim_eff}" velocity="${lim_vel}"/><!--
+            <limit effort="${lim_eff}" lower="${lim_low_1}" upper="${lim_up_1}" velocity="${lim_vel}"/>-->
         </joint>
         <link name="link1">
@@ -84,12 +98,12 @@
                 <origin rpy="0 0 0" xyz="0 0 0"/>
                 <geometry>
-                    <mesh filename="package://rover_arm/meshes/Link1.dae"/>
+                    <mesh filename="package://rover_arm/meshes/Coll_Link1.stl"/>
                 </geometry>
                 <material name="black"/>
             </visual>
             <inertial>
-                <origin rpy="0 0 0" xyz="0 0 ${link1_len/2}"/>
-                <mass value="1"/>
-                <box_inertia m="1" x="${link1_width}" y="${link1_width}" z="${link1_len}" />
+                <origin rpy="0 0 0" xyz="${link1_com}"/>
+                <mass value="${link1_mass}"/>
+                <box_inertia m="${link1_mass}" x="${link1_width}" y="${link1_width}" z="${link1_len}" />
             </inertial>
         </link>
@@ -112,12 +126,12 @@
                 <origin rpy="0 0 0" xyz="0 0 0"/>
                 <geometry>
-                    <mesh filename="package://rover_arm/meshes/Link2.dae"/>
+                    <mesh filename="package://rover_arm/meshes/Coll_Link2.stl"/>
                 </geometry>
                 <material name="orange"/>
             </visual>
             <inertial>
-                <origin rpy="0 0 0" xyz="0 0 ${link2_len/2}"/>
-                <mass value="1"/>
-                <box_inertia m="1" x="${link2_width}" y="${link2_width}" z="${link2_len}" />
+                <origin rpy="0 0 0" xyz="${link2_com}"/>
+                <mass value="${link2_mass}"/>
+                <box_inertia m="${link2_mass}" x="${link2_width}" y="${link2_width}" z="${link2_len}" />
             </inertial>
         </link>
@@ -139,7 +153,7 @@
             </visual>
             <inertial>
-                <origin rpy="0 0 0" xyz="0 0 0"/>
-                <mass value="1"/>
-                <box_inertia m="1" x="${link3_width}" y="${link3_width}" z="${link3_len}" />
+                <origin rpy="0 0 0" xyz="${link3_com}"/>
+                <mass value="${link3_mass}"/>
+                <box_inertia m="${link3_mass}" x="${link3_width}" y="${link3_width}" z="${link3_len}" />
             </inertial>
         </link>
@@ -161,7 +175,7 @@
             </visual>
             <inertial>
-                <origin rpy="0 0 0" xyz="0 0 0"/>
-                <mass value="1"/>
-                <box_inertia m="1" x="${link4_width}" y="${link4_width}" z="${link4_len}" />
+                <origin rpy="0 0 0" xyz="${link4_com}"/>
+                <mass value="${link4_mass}"/>
+                <box_inertia m="${link4_mass}" x="${link4_width}" y="${link4_width}" z="${link4_len}" />
             </inertial>
         </link>
@@ -184,12 +198,12 @@
                 <origin rpy="0 0 0" xyz="0 0 0"/>
                 <geometry>
-                    <mesh filename="package://rover_arm/meshes/Hand.dae"/>
+                    <mesh filename="package://rover_arm/meshes/Coll_Hand.stl"/>
                 </geometry>
                 <material name="black"/>
             </visual>
             <inertial>
-                <origin rpy="0 0 0" xyz="0 0 ${link5_len/2}"/>
-                <mass value="1"/>
-                <box_inertia m="1" x="${link5_width}" y="${link5_width}" z="${link5_len}" />
+                <origin rpy="0 0 0" xyz="${link_hand_com}"/>
+                <mass value="${link_hand_mass}"/>
+                <box_inertia m="${link_hand_mass}" x="${link5_width}" y="${link5_width}" z="${link5_len}" />
             </inertial>
         </link>

File: urdf/testarm.xacro (robot description, xacro)
@@ -22,5 +22,5 @@
       </inertial>
     </link>
-    <arm parent="base_link" translateX="0.3" translateY="0" translateZ="0.05"/>
+    <arm parent="base_link" translateX="0" translateY="0.3" translateZ="0.15"/>
     <!--   base link can't have inertia   -->
     <link name="world" />

Commit message: Use the correct mesh for visual

File: urdf/arm.xacro (robot description, xacro)
@@ -55,5 +55,5 @@
             <parent link="${parent}"/>
             <child link="link0"/>
-            <origin rpy="0 0 0" xyz="${translateX} ${translateY} ${translateZ}"/>
+            <origin rpy="-1.6 0 0" xyz="${translateX} ${translateY} ${translateZ}"/>
             <axis xyz="0 0 1"/>
             <limit effort="${lim_eff}" velocity="${lim_vel}"/>
@@ -69,5 +69,5 @@
                 <origin rpy="0 0 0" xyz="0 0 0"/>
                 <geometry>
-                    <mesh filename="package://rover_arm/meshes/Coll_Link0.stl"/>
+                    <mesh filename="package://rover_arm/meshes/Link0.dae"/>
                 </geometry>
                 <material name="orange"/>
@@ -98,5 +98,5 @@
                 <origin rpy="0 0 0" xyz="0 0 0"/>
                 <geometry>
-                    <mesh filename="package://rover_arm/meshes/Coll_Link1.stl"/>
+                    <mesh filename="package://rover_arm/meshes/Link1.dae"/>
                 </geometry>
                 <material name="black"/>
@@ -126,5 +126,5 @@
                 <origin rpy="0 0 0" xyz="0 0 0"/>
                 <geometry>
-                    <mesh filename="package://rover_arm/meshes/Coll_Link2.stl"/>
+                    <mesh filename="package://rover_arm/meshes/Link2.dae"/>
                 </geometry>
                 <material name="orange"/>
@@ -198,5 +198,5 @@
                 <origin rpy="0 0 0" xyz="0 0 0"/>
                 <geometry>
-                    <mesh filename="package://rover_arm/meshes/Coll_Hand.stl"/>
+                    <mesh filename="package://rover_arm/meshes/Hand.dae"/>
                 </geometry>
                 <material name="black"/>
