Commit message: renamed base_cylinder due to name conflict with rover.xacro

File: urdf/testarm.xacro (robot description, xacro)
@@ -2,5 +2,5 @@
 <robot name="testarm" xmlns:xacro="http://www.ros.org/wiki/xacro">
     <xacro:include filename="$(find rover_arm)/urdf/arm.xacro"/>
-    <link name="base_link">
+    <link name="base_cylinder">
       <collision>
         <origin rpy="0 0 0" xyz="0.0 0.0 0.0"/>
@@ -22,10 +22,10 @@
       </inertial>
     </link>
-    <arm parent="base_link" translateX="0" translateY="0.3" translateZ="0.15"/>
+    <arm parent="base_cylinder" translateX="0" translateY="0.3" translateZ="0.15"/>
     <!--   base link can't have inertia   -->
     <link name="world" />
     <joint name="world_joint" type="fixed">
         <parent link="world" />
-        <child link = "base_link" />
+        <child link = "base_cylinder" />
         <origin xyz="0.0 0.0 0.0" rpy="0.0 0.0 0.0" />
     </joint>

Commit message: arm control on rover works now

File: urdf/testarm.xacro (robot description, xacro)
@@ -24,6 +24,7 @@
     <arm parent="base_cylinder" translateX="0" translateY="0.3" translateZ="0.15"/>
     <!--   base link can't have inertia   -->
+    <!--   MoveIt needs a fixed world joint   -->
     <link name="world" />
-    <joint name="world_joint" type="fixed">
+    <joint name="world_joint" type="continuous">
         <parent link="world" />
         <child link = "base_cylinder" />
@@ -33,4 +34,5 @@
       <plugin name="joint_state_publisher" filename="libgazebo_ros_joint_state_publisher.so">
          <jointName>
+<!--             world_joint, -->
             joint0,
             joint1,
