Commit message: better joint limits and launch file configs

File: urdf/carm.xacro (robot description, xacro)
@@ -31,11 +31,13 @@
     <xacro:property name="offset_gripper" value="0.01" />
     <xacro:property name="lim_eff" value="3000" />
-    <xacro:property name="lim_low_1" value="${-pi * 1/3}" />
-    <xacro:property name="lim_up_1" value="${pi * 2/3}" />
-    <xacro:property name="lim_low_2" value="-2.9698" />
-    <xacro:property name="lim_up_2" value="1.18" />
-    <xacro:property name="lim_low_4" value="${-pi/2}" />
-    <xacro:property name="lim_up_4" value="${pi/2}" />
     <xacro:property name="lim_vel" value="1.571" />
+    <xacro:property name="lim_low_1" value="-0.4" />
+    <xacro:property name="lim_up_1" value="${pi * 1}" />
+    <xacro:property name="lim_low_2" value="-0.1" />
+    <xacro:property name="lim_up_2" value="${pi}" />
+    <xacro:property name="lim_low_3" value="${-pi * 2/3}" />
+    <xacro:property name="lim_up_3" value="${pi * 2/3}" />
+    <xacro:property name="lim_low_gripper" value="0" />
+    <xacro:property name="lim_up_gripper" value="0.04" />
     <xacro:property name="M_PI" value="3.1415926535897931" />
     <xacro:property name="M_PI_2" value="1.570796327" />
@@ -82,11 +84,10 @@
         </link>
         <!--  Link 1: up/down arm segment 1  -->
-        <joint name="joint1" type="continuous">
+        <joint name="joint1" type="revolute">
             <parent link="link0"/>
             <child link="link1"/>
                 <origin rpy="0 0 0" xyz="0 0 0.037"/>
             <axis xyz="1 0 0"/>
-            <limit effort="${lim_eff}" velocity="${lim_vel}"/><!--
-            <limit effort="${lim_eff}" lower="${lim_low_1}" upper="${lim_up_1}" velocity="${lim_vel}"/>-->
+            <limit effort="${lim_eff}" lower="${lim_low_1}" upper="${lim_up_1}" velocity="${lim_vel}"/>
         </joint>
         <link name="link1">
@@ -139,10 +140,10 @@
         </link>
         <!--  Link 3: swivel up/down  -->
-        <joint name="joint3" type="continuous">
+        <joint name="joint3" type="revolute">
             <parent link="link2"/>
             <child link="link3"/>
                 <origin rpy="0 0 0" xyz="0 0.182 0"/>
             <axis xyz="1 0 0"/>
-            <limit effort="${lim_eff}" velocity="${lim_vel}"/>
+            <limit effort="${lim_eff}" lower="${lim_low_3}" upper="${lim_up_3}" velocity="${lim_vel}"/>
         </joint>
         <link name="link3">
@@ -194,5 +195,5 @@
                 <origin rpy="0 0 0" xyz="-0.043 0.032 0"/>
             <axis xyz="1 0 0"/>
-            <limit effort="${lim_eff}" lower="${lim_low_2}" upper="${lim_up_2}" velocity="${lim_vel}"/>
+            <limit effort="${lim_eff}" lower="${lim_low_gripper}" upper="${lim_up_gripper}" velocity="${lim_vel}"/>
         </joint>
         <link name="link_gripper_a">
@@ -219,7 +220,7 @@
             <parent link="link_hand"/>
             <child link="link_gripper_b"/>
-                <origin rpy="0 0 0" xyz="0.043 0.032 0"/>
-            <axis xyz="1 0 0"/>
-            <limit effort="${lim_eff}" lower="${lim_low_2}" upper="${lim_up_2}" velocity="${lim_vel}"/>
+                <origin rpy="0 ${pi} 0" xyz="0.043 0.032 0"/>
+            <axis xyz="1 0 0"/>
+            <limit effort="${lim_eff}" lower="${lim_low_gripper}" upper="${lim_up_gripper}" velocity="${lim_vel}"/>
         </joint>
         <link name="link_gripper_b">
