Commit message: competition arm location

File: urdf/rover_with_carm.xacro (robot description, xacro)
@@ -14,5 +14,5 @@
     <!--   fix arm direction and position on the rover   -->
     <joint name="arm_body_connection" type="fixed">
-            <origin xyz="0.2 0.0 0.17" rpy="${M_PI_2} 0 ${-M_PI_2}"/>
+            <origin xyz="0.48 0.0 0.21" rpy="${M_PI_2} 0 ${-M_PI_2}"/>
             <parent link="chassis"/>
             <child link="arm_body_base"/>
